File: Z80_SBC.kicad_sch (KiCad schematic)
At the start: 38 parts, among them J1 USB_C_Receptacle_PowerOnly_6P, J2 Conn_01x04_Pin, SW1 SW_Push, U1 Z80CPU, U2 HM62256BLP, U3 27C64, U4 74HCT04, U5 74LS139, U6 MC68A50, U7 74LS573, U8 74LS32, Y1 1.8432MHz

Commit message: minor fixes
Parts:
- added C12: 0.1uF, Capacitor_THT:C_Radial_D4.0mm_H5.0mm_P1.50mm, symbol Device:C_Small
- R4: value 3k3 -> 10k
Connections:
- net 5V: now also C4.1
- net GND: now also C12.2; no longer U4.8, U5.10 (O2), U5.11 (O1), U5.12 (O0), U5.9 (O3), U8.3, U8.6
- net at R3.2, SW1.2, U1.26 (~{RESET}): now also C12.1; no longer C4.1
Other:
- moved on the sheet: C4
Changed lines of the file:
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@@
   (junction (at 251.46 158.75) (diameter 0) (color 0 0 0 0)
   )
-  (junction (at 144.78 190.5) (diameter 0) (color 0 0 0 0)
-  )
-  (junction (at 152.4 184.15) (diameter 0) (color 0 0 0 0)
-  )
   (junction (at 238.76 158.75) (diameter 0) (color 0 0 0 0)
   )
@@
   (junction (at 219.71 149.86) (diameter 0) (color 0 0 0 0)
   )
-  (junction (at 232.41 149.86) (diameter 0) (color 0 0 0 0)
+  (junction (at 24.13 27.94) (diameter 0) (color 0 0 0 0)
   )
-  (junction (at 106.68 185.42) (diameter 0) (color 0 0 0 0)
+  (junction (at 232.41 149.86) (diameter 0) (color 0 0 0 0)
   )
   (junction (at 134.62 151.13) (diameter 0) (color 0 0 0 0)
@@
   (junction (at 232.41 158.75) (diameter 0) (color 0 0 0 0)
   )
-  (junction (at 106.68 187.96) (diameter 0) (color 0 0 0 0)
-  )
   (junction (at 238.76 149.86) (diameter 0) (color 0 0 0 0)
   )
   (junction (at 226.06 158.75) (diameter 0) (color 0 0 0 0)
   )
-  (junction (at 106.68 190.5) (diameter 0) (color 0 0 0 0)
-  )
   (junction (at 154.94 119.38) (diameter 0) (color 0 0 0 0)
   )
@@
     (stroke (width 0) (type default))
   )
-  (wire (pts (xy 106.68 185.42) (xy 106.68 187.96))
-    (stroke (width 0) (type default))
-  )
   (wire (pts (xy 149.86 146.05) (xy 152.4 146.05))
     (stroke (width 0) (type default))
@@
     (stroke (width 0) (type default))
   )
-  (wire (pts (xy 106.68 187.96) (xy 106.68 190.5))
-    (stroke (width 0) (type default))
-  )
   (bus (pts (xy 154.94 107.95) (xy 154.94 110.49))
     (stroke (width 0) (type default))
@@
     (stroke (width 0) (type default))
   )
-  (wire (pts (xy 22.86 33.02) (xy 22.86 38.1))
-    (stroke (width 0) (type default))
-  )
   (bus (pts (xy 154.94 119.38) (xy 219.71 119.38))
     (stroke (width 0) (type default))
@@
     (stroke (width 0) (type default))
   )
-  (wire (pts (xy 152.4 170.18) (xy 152.4 184.15))
-    (stroke (width 0) (type default))
-  )
   (wire (pts (xy 24.13 118.11) (xy 24.13 129.54))
     (stroke (width 0) (type default))
@@
     (stroke (width 0) (type default))
   )
-  (wire (pts (xy 22.86 27.94) (xy 33.02 27.94))
+  (wire (pts (xy 33.02 52.07) (xy 22.86 52.07))
     (stroke (width 0) (type default))
   )
-  (wire (pts (xy 33.02 52.07) (xy 22.86 52.07))
+  (wire (pts (xy 22.86 27.94) (xy 24.13 27.94))
     (stroke (width 0) (type default))
   )
@@
     (stroke (width 0) (type default))
   )
-  (wire (pts (xy 152.4 190.5) (xy 144.78 190.5))
-    (stroke (width 0) (type default))
-  )
   (wire (pts (xy 271.78 129.54) (xy 271.78 132.08))
     (stroke (width 0) (type default))
@@
     (stroke (width 0) (type default))
   )
-  (wire (pts (xy 144.78 190.5) (xy 137.16 190.5))
-    (stroke (width 0) (type default))
-  )
   (wire (pts (xy 120.65 110.49) (xy 123.19 110.49))
     (stroke (width 0) (type default))
@@
     (stroke (width 0) (type default))
   )
-  (wire (pts (xy 22.86 38.1) (xy 19.05 38.1))
+  (wire (pts (xy 24.13 38.1) (xy 19.05 38.1))
     (stroke (width 0) (type default))
   )
@@
     (stroke (width 0) (type default))
   )
+  (wire (pts (xy 24.13 35.56) (xy 24.13 38.1))
+    (stroke (width 0) (type default))
+  )
   (bus (pts (xy 219.71 106.68) (xy 219.71 109.22))
     (stroke (width 0) (type default))
@@
     (stroke (width 0) (type default))
   )
-  (wire (pts (xy 120.65 151.13) (xy 134.62 151.13))
+  (wire (pts (xy 24.13 27.94) (xy 33.02 27.94))
     (stroke (width 0) (type default))
   )
-  (wire (pts (xy 106.68 182.88) (xy 106.68 185.42))
+  (wire (pts (xy 120.65 151.13) (xy 134.62 151.13))
     (stroke (width 0) (type default))
   )
@@
     (stroke (width 0) (type default))
   )
-  (wire (pts (xy 152.4 184.15) (xy 152.4 190.5))
-    (stroke (width 0) (type default))
-  )
   (wire (pts (xy 148.59 113.03) (xy 152.4 113.03))
     (stroke (width 0) (type default))
@@
     (stroke (width 0) (type default))
   )
-  (wire (pts (xy 144.78 190.5) (xy 144.78 191.77))
-    (stroke (width 0) (type default))
-  )
   (wire (pts (xy 120.65 130.81) (xy 123.19 130.81))
     (stroke (width 0) (type default))
@@
     (stroke (width 0) (type default))
   )
+  (wire (pts (xy 24.13 30.48) (xy 24.13 27.94))
+    (stroke (width 0) (type default))
+  )
   (wire (pts (xy 148.59 102.87) (xy 152.4 102.87))
     (stroke (width 0) (type default))
@@
     )
   )
-  (symbol (lib_id "Device:C_Small") (at 22.86 30.48 0) (unit 1)
+  (symbol (lib_id "Device:C_Small") (at 226.06 153.67 0) (unit 1)
     (in_bom yes) (on_board yes) (dnp no)
-    (property "Reference" "C4" (at 24.13 33.02 0)
+    (property "Reference" "C4" (at 227.33 157.48 90)
       (effects (font (size 1.27 1.27)) (justify left))
     )
-    (property "Value" "0.1uF" (at 24.13 29.21 0)
+    (property "Value" "0.1uF" (at 223.52 157.48 90)
       (effects (font (size 1.27 1.27)) (justify left))
     )
-    (property "Footprint" "Capacitor_THT:C_Radial_D4.0mm_H5.0mm_P1.50mm" (at 22.86 30.48 0)
+    (property "Footprint" "Capacitor_THT:C_Radial_D4.0mm_H5.0mm_P1.50mm" (at 226.06 153.67 0)
       (effects (font (size 1.27 1.27)) hide)
     )
-    (property "Datasheet" "~" (at 22.86 30.48 0)
+    (property "Datasheet" "~" (at 226.06 153.67 0)
       (effects (font (size 1.27 1.27)) hide)
     )
@@
       (effects (font (size 1.27 1.27)) (justify left))
     )
-    (property "Value" "3k3" (at 16.51 52.07 90)
+    (property "Value" "10k" (at 16.51 52.07 90)
       (effects (font (size 1.27 1.27)) (justify left))
     )
@@
     )
   )
-  (symbol (lib_id "power:GND") (at 128.27 189.23 0) (unit 1)
-    (in_bom yes) (on_board yes) (dnp no) (fields_autoplaced)
-    (property "Reference" "#PWR08" (at 128.27 195.58 0)
-      (effects (font (size 1.27 1.27)) hide)
-    )
-    (property "Value" "GND" (at 128.27 194.31 0)
-      (effects (font (size 1.27 1.27)))
-    )
-    (property "Footprint" "" (at 128.27 189.23 0)
-      (effects (font (size 1.27 1.27)) hide)
-    )
-    (property "Datasheet" "" (at 128.27 189.23 0)
-      (effects (font (size 1.27 1.27)) hide)
-    )
-    (pin "1")
-    (instances
-      (project "Z80_SBC"
-        (path "/6573ed54-b921-4c04-b990-e84729c40c2c"
-          (reference "#PWR08") (unit 1)
-        )
-      )
-    )
-  )
   (symbol (lib_id "Device:C_Small") (at 245.11 153.67 0) (unit 1)
     (in_bom yes) (on_board yes) (dnp no)
@@
     )
   )
-  (symbol (lib_id "power:GND") (at 144.78 191.77 0) (unit 1)
+  (symbol (lib_id "power:GND") (at 137.16 190.5 0) (unit 1)
     (in_bom yes) (on_board yes) (dnp no) (fields_autoplaced)
-    (property "Reference" "#PWR014" (at 144.78 198.12 0)
+    (property "Reference" "#PWR014" (at 137.16 196.85 0)
       (effects (font (size 1.27 1.27)) hide)
     )
-    (property "Value" "GND" (at 144.78 196.85 0)
+    (property "Value" "GND" (at 137.16 195.58 0)
       (effects (font (size 1.27 1.27)))
     )
-    (property "Footprint" "" (at 144.78 191.77 0)
+    (property "Footprint" "" (at 137.16 190.5 0)
       (effects (font (size 1.27 1.27)) hide)
     )
-    (property "Datasheet" "" (at 144.78 191.77 0)
+    (property "Datasheet" "" (at 137.16 190.5 0)
       (effects (font (size 1.27 1.27)) hide)
     )
@@
     )
   )
+  (symbol (lib_id "Device:C_Small") (at 24.13 33.02 0) (unit 1)
+    (in_bom yes) (on_board yes) (dnp no)
+    (property "Reference" "C12" (at 25.4 35.56 0)
+      (effects (font (size 1.27 1.27)) (justify left))
+    )
+    (property "Value" "0.1uF" (at 25.4 31.75 0)
+      (effects (font (size 1.27 1.27)) (justify left))
+    )
+    (property "Footprint" "Capacitor_THT:C_Radial_D4.0mm_H5.0mm_P1.50mm" (at 24.13 33.02 0)
+      (effects (font (size 1.27 1.27)) hide)
+    )
+    (property "Datasheet" "~" (at 24.13 33.02 0)
+      (effects (font (size 1.27 1.27)) hide)
+    )
+    (pin "1")
+    (pin "2")
+    (instances
+      (project "Z80_SBC"
+        (path "/6573ed54-b921-4c04-b990-e84729c40c2c"
+          (reference "C12") (unit 1)
+        )
+      )
+    )
+  )
   (symbol (lib_id "74xx:74LS573") (at 238.76 106.68 0) (unit 1)
     (in_bom yes) (on_board yes) (dnp no) (fields_autoplaced)
@@
         )
       )
-    )
-  )
-  (symbol (lib_id "power:GND") (at 106.68 190.5 0) (unit 1)
-    (in_bom yes) (on_board yes) (dnp no) (fields_autoplaced)
-    (property "Reference" "#PWR06" (at 106.68 196.85 0)
-      (effects (font (size 1.27 1.27)) hide)
-    )
-    (property "Value" "GND" (at 106.68 195.58 0)
-      (effects (font (size 1.27 1.27)))
-    )
-    (property "Footprint" "" (at 106.68 190.5 0)
-      (effects (font (size 1.27 1.27)) hide)
-    )
-    (property "Datasheet" "" (at 106.68 190.5 0)
-      (effects (font (size 1.27 1.27)) hide)
-    )
-    (pin "1")
-    (instances
-      (project "Z80_SBC"
-        (path "/6573ed54-b921-4c04-b990-e84729c40c2c"
-          (reference "#PWR06") (unit 1)
-        )
-      )
